File: Nanobuino/Eagle/Nanobuino/Nanobuino.sch (EAGLE design)
At the start: 2 parts, among them J1 HEAD15-NOSS, J2 HEAD15-NOSS-1

Commit message: Lots of parts added to schematic
Parts:
- added IC1: MCP73833-UN, adafruit:MCP73833-UN
- added SP1: SPEAKER/AL60P, adafruit:SPEAKER/AL60P
- added SW1, SW2, SW3, SW4, SW5, SW6, SW7: SPST_TACT-EVQQ2, adafruit:SPST_TACT-EVQQ2
- added T1: (no value), transistor-neu-to92:MMBT2222ALT1-NPN-SOT23-BEC
- added X1: STEREOJACK, adafruit:STEREOJACK
Changed lines of the file:
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@@
 <layer number="54" name="bGND_GNDA" color="1" fill="9" visible="no" active="no"/>
 <layer number="56" name="wert" color="7" fill="1" visible="no" active="no"/>
+<layer number="57" name="tCAD" color="7" fill="1" visible="no" active="no"/>
 <layer number="91" name="Nets" color="2" fill="1" visible="yes" active="yes"/>
 <layer number="92" name="Busses" color="1" fill="1" visible="yes" active="yes"/>
@@
 <layer number="101" name="Patch_Top" color="12" fill="4" visible="yes" active="yes"/>
 <layer number="102" name="Vscore" color="7" fill="1" visible="yes" active="yes"/>
+<layer number="103" name="fp3" color="7" fill="1" visible="no" active="yes"/>
 <layer number="104" name="Name" color="7" fill="1" visible="yes" active="yes"/>
+<layer number="105" name="Beschreib" color="9" fill="1" visible="yes" active="yes"/>
+<layer number="106" name="BGA-Top" color="4" fill="1" visible="yes" active="yes"/>
+<layer number="107" name="BD-Top" color="5" fill="1" visible="yes" active="yes"/>
+<layer number="108" name="fp8" color="7" fill="1" visible="no" active="yes"/>
+<layer number="109" name="fp9" color="7" fill="1" visible="no" active="yes"/>
+<layer number="110" name="fp0" color="7" fill="1" visible="no" active="yes"/>
+<layer number="111" name="LPC17xx" color="7" fill="1" visible="yes" active="yes"/>
+<layer number="112" name="tSilk" color="7" fill="1" visible="yes" active="yes"/>
 <layer number="116" name="Patch_BOT" color="9" fill="4" visible="yes" active="yes"/>
 <layer number="121" name="_tsilk" color="7" fill="1" visible="yes" active="yes"/>
 <layer number="122" name="_bsilk" color="7" fill="1" visible="yes" active="yes"/>
+<layer number="123" name="tTestmark" color="7" fill="1" visible="no" active="yes"/>
+<layer number="124" name="bTestmark" color="7" fill="1" visible="no" active="yes"/>
+<layer number="125" name="_tNames" color="7" fill="1" visible="yes" active="yes"/>
+<layer number="126" name="_bNames" color="7" fill="1" visible="yes" active="yes"/>
+<layer number="127" name="_tValues" color="7" fill="1" visible="yes" active="yes"/>
+<layer number="128" name="_bValues" color="7" fill="1" visible="yes" active="yes"/>
+<layer number="131" name="tAdjust" color="7" fill="1" visible="no" active="yes"/>
+<layer number="132" name="bAdjust" color="7" fill="1" visible="no" active="yes"/>
+<layer number="144" name="Drill_legend" color="7" fill="1" visible="yes" active="yes"/>
+<layer number="150" name="Notes" color="7" fill="1" visible="no" active="yes"/>
 <layer number="151" name="HeatSink" color="7" fill="1" visible="yes" active="yes"/>
+<layer number="152" name="_bDocu" color="7" fill="1" visible="yes" active="yes"/>
+<layer number="153" name="FabDoc1" color="6" fill="1" visible="no" active="no"/>
+<layer number="154" name="FabDoc2" color="2" fill="1" visible="no" active="no"/>
+<layer number="155" name="FabDoc3" color="7" fill="15" visible="no" active="no"/>
+<layer number="199" name="Contour" color="7" fill="1" visible="yes" active="yes"/>
 <layer number="200" name="200bmp" color="1" fill="10" visible="no" active="no"/>
 <layer number="201" name="201bmp" color="2" fill="1" visible="no" active="no"/>
 <layer number="202" name="202bmp" color="3" fill="1" visible="no" active="no"/>
+<layer number="203" name="203bmp" color="4" fill="10" visible="yes" active="yes"/>
+<layer number="204" name="204bmp" color="5" fill="10" visible="yes" active="yes"/>
+<layer number="205" name="205bmp" color="6" fill="10" visible="yes" active="yes"/>
+<layer number="206" name="206bmp" color="7" fill="10" visible="yes" active="yes"/>
+<layer number="207" name="207bmp" color="8" fill="10" visible="yes" active="yes"/>
+<layer number="208" name="208bmp" color="9" fill="10" visible="yes" active="yes"/>
+<layer number="209" name="209bmp" color="7" fill="1" visible="no" active="yes"/>
+<layer number="210" name="210bmp" color="7" fill="1" visible="no" active="yes"/>
+<layer number="211" name="211bmp" color="7" fill="1" visible="yes" active="yes"/>
+<layer number="212" name="212bmp" color="7" fill="1" visible="yes" active="yes"/>
+<layer number="213" name="213bmp" color="7" fill="1" visible="yes" active="yes"/>
+<layer number="214" name="214bmp" color="7" fill="1" visible="yes" active="yes"/>
+<layer number="215" name="215bmp" color="7" fill="1" visible="yes" active="yes"/>
+<layer number="216" name="216bmp" color="7" fill="1" visible="yes" active="yes"/>
+<layer number="217" name="217bmp" color="18" fill="1" visible="no" active="no"/>
+<layer number="218" name="218bmp" color="19" fill="1" visible="no" active="no"/>
+<layer number="219" name="219bmp" color="20" fill="1" visible="no" active="no"/>
+<layer number="220" name="220bmp" color="21" fill="1" visible="no" active="no"/>
+<layer number="221" name="221bmp" color="22" fill="1" visible="no" active="no"/>
+<layer number="222" name="222bmp" color="23" fill="1" visible="no" active="no"/>
+<layer number="223" name="223bmp" color="24" fill="1" visible="no" active="no"/>
+<layer number="224" name="224bmp" color="25" fill="1" visible="no" active="no"/>
+<layer number="248" name="Housing" color="7" fill="1" visible="yes" active="yes"/>
+<layer number="249" name="Edge" color="7" fill="1" visible="yes" active="yes"/>
 <layer number="250" name="Descript" color="3" fill="1" visible="no" active="no"/>
 <layer number="251" name="SMDround" color="12" fill="11" visible="no" active="no"/>
@@
 <part name="J1" library="MyCON2" deviceset="HEAD15-NOSS" device=""/>
 <part name="J2" library="MyCON2" deviceset="HEAD15-NOSS-1" device=""/>
+<part name="X1" library="adafruit" deviceset="STEREOJACK" device=""/>
+<part name="SP1" library="adafruit" deviceset="SPEAKER" device="/AL60P"/>
+<part name="SW1" library="adafruit" deviceset="SPST_TACT" device="-EVQQ2"/>
+<part name="SW2" library="adafruit" deviceset="SPST_TACT" device="-EVQQ2"/>
+<part name="SW3" library="adafruit" deviceset="SPST_TACT" device="-EVQQ2"/>
+<part name="SW4" library="adafruit" deviceset="SPST_TACT" device="-EVQQ2"/>
+<part name="SW5" library="adafruit" deviceset="SPST_TACT" device="-EVQQ2"/>
+<part name="SW6" library="adafruit" deviceset="SPST_TACT" device="-EVQQ2"/>
+<part name="SW7" library="adafruit" deviceset="SPST_TACT" device="-EVQQ2"/>
+<part name="IC1" library="adafruit" deviceset="MCP73833" device="-UN"/>
+<part name="T1" library="transistor-neu-to92" deviceset="*-NPN-" device="SOT23-BEC" technology="MMBT2222ALT1"/>
 </parts>
 <sheets>
@@
 <instance part="J1" gate="G$1" x="60.96" y="45.72" rot="MR0"/>
 <instance part="J2" gate="G$1" x="86.36" y="45.72"/>
+<instance part="X1" gate="1" x="43.18" y="93.98"/>
+<instance part="SP1" gate="S1" x="71.12" y="104.14" rot="MR180"/>
+<instance part="SW1" gate="G$1" x="45.72" y="5.08" rot="MR180"/>
+<instance part="SW2" gate="G$1" x="66.04" y="2.54" rot="MR180"/>
+<instance part="SW3" gate="G$1" x="86.36" y="2.54" rot="MR180"/>
+<instance part="SW4" gate="G$1" x="104.14" y="2.54" rot="MR180"/>
+<instance part="SW5" gate="G$1" x="119.38" y="2.54" rot="MR180"/>
+<instance part="SW6" gate="G$1" x="142.24" y="2.54" rot="MR180"/>
+<instance part="SW7" gate="G$1" x="160.02" y="2.54" rot="MR180"/>
+<instance part="IC1" gate="G$1" x="149.86" y="76.2"/>
+<instance part="T1" gate="G$1" x="154.94" y="38.1"/>
 </instances>
 <busses>

Commit message: 1st layout
Parts:
- added JP1_LCD: (no value), adafruit:PINHD-1X8CLEANBIG
- added POT1: THUMBPOT, adafruit:THUMBPOT
- added S1_POWER: EG1213, adafruit:EG1213
- added U$20: MICROSD, adafruit:MICROSD
- renumbered SW1 to SW1UP, SW2 to SW2RIGHT, SW3 to SW3DOWN, SW4 to SW4LEFT, SW5 to SW5ABTN, SW6 to SW6BBTN, SW7 to SW7CBTN
Connections:
- net COM: now also SW1UP.S, SW1UP.S1, SW2RIGHT.S, SW2RIGHT.S1, SW3DOWN.S, SW3DOWN.S1, SW4LEFT.S, SW4LEFT.S1, SW5ABTN.S, SW5ABTN.S1, SW6BBTN.S, SW6BBTN.S1, SW7CBTN.S, SW7CBTN.S1
Changed lines of the file:
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@@
 <part name="X1" library="adafruit" deviceset="STEREOJACK" device=""/>
 <part name="SP1" library="adafruit" deviceset="SPEAKER" device="/AL60P"/>
-<part name="SW1" library="adafruit" deviceset="SPST_TACT" device="-EVQQ2"/>
-<part name="SW2" library="adafruit" deviceset="SPST_TACT" device="-EVQQ2"/>
-<part name="SW3" library="adafruit" deviceset="SPST_TACT" device="-EVQQ2"/>
-<part name="SW4" library="adafruit" deviceset="SPST_TACT" device="-EVQQ2"/>
-<part name="SW5" library="adafruit" deviceset="SPST_TACT" device="-EVQQ2"/>
-<part name="SW6" library="adafruit" deviceset="SPST_TACT" device="-EVQQ2"/>
-<part name="SW7" library="adafruit" deviceset="SPST_TACT" device="-EVQQ2"/>
+<part name="SW1UP" library="adafruit" deviceset="SPST_TACT" device="-EVQQ2"/>
+<part name="SW2RIGHT" library="adafruit" deviceset="SPST_TACT" device="-EVQQ2"/>
+<part name="SW3DOWN" library="adafruit" deviceset="SPST_TACT" device="-EVQQ2"/>
+<part name="SW4LEFT" library="adafruit" deviceset="SPST_TACT" device="-EVQQ2"/>
+<part name="SW5ABTN" library="adafruit" deviceset="SPST_TACT" device="-EVQQ2"/>
+<part name="SW6BBTN" library="adafruit" deviceset="SPST_TACT" device="-EVQQ2"/>
+<part name="SW7CBTN" library="adafruit" deviceset="SPST_TACT" device="-EVQQ2"/>
 <part name="IC1" library="adafruit" deviceset="MCP73833" device="-UN"/>
 <part name="T1" library="transistor-neu-to92" deviceset="*-NPN-" device="SOT23-BEC" technology="MMBT2222ALT1"/>
+<part name="U$3" library="MyPOW" deviceset="COM" device=""/>
+<part name="U$4" library="MyPOW" deviceset="COM" device=""/>
+<part name="U$5" library="MyPOW" deviceset="COM" device=""/>
+<part name="U$9" library="MyPOW" deviceset="COM" device=""/>
+<part name="U$10" library="MyPOW" deviceset="COM" device=""/>
+<part name="U$11" library="MyPOW" deviceset="COM" device=""/>
+<part name="U$12" library="MyPOW" deviceset="COM" device=""/>
+<part name="U$13" library="MyPOW" deviceset="COM" device=""/>
+<part name="U$14" library="MyPOW" deviceset="COM" device=""/>
+<part name="U$15" library="MyPOW" deviceset="COM" device=""/>
+<part name="U$16" library="MyPOW" deviceset="COM" device=""/>
+<part name="U$17" library="MyPOW" deviceset="COM" device=""/>
+<part name="U$18" library="MyPOW" deviceset="COM" device=""/>
+<part name="U$19" library="MyPOW" deviceset="COM" device=""/>
+<part name="JP1_LCD" library="adafruit" deviceset="PINHD-1X8" device="CLEANBIG"/>
+<part name="U$20" library="adafruit" deviceset="MICROSD" device=""/>
+<part name="POT1" library="adafruit" deviceset="THUMBPOT" device=""/>
+<part name="S1_POWER" library="adafruit" deviceset="EG1213" device=""/>
 </parts>
 <sheets>
@@
 <instance part="X1" gate="1" x="43.18" y="93.98"/>
 <instance part="SP1" gate="S1" x="71.12" y="104.14" rot="MR180"/>
-<instance part="SW1" gate="G$1" x="45.72" y="5.08" rot="MR180"/>
-<instance part="SW2" gate="G$1" x="66.04" y="2.54" rot="MR180"/>
-<instance part="SW3" gate="G$1" x="86.36" y="2.54" rot="MR180"/>
-<instance part="SW4" gate="G$1" x="104.14" y="2.54" rot="MR180"/>
-<instance part="SW5" gate="G$1" x="119.38" y="2.54" rot="MR180"/>
-<instance part="SW6" gate="G$1" x="142.24" y="2.54" rot="MR180"/>
-<instance part="SW7" gate="G$1" x="160.02" y="2.54" rot="MR180"/>
+<instance part="SW1UP" gate="G$1" x="45.72" y="5.08" rot="MR180"/>
+<instance part="SW2RIGHT" gate="G$1" x="66.04" y="2.54" rot="MR180"/>
+<instance part="SW3DOWN" gate="G$1" x="86.36" y="2.54" rot="MR180"/>
+<instance part="SW4LEFT" gate="G$1" x="104.14" y="2.54" rot="MR180"/>
+<instance part="SW5ABTN" gate="G$1" x="119.38" y="2.54" rot="MR180"/>
+<instance part="SW6BBTN" gate="G$1" x="142.24" y="2.54" rot="MR180"/>
+<instance part="SW7CBTN" gate="G$1" x="160.02" y="2.54" rot="MR180"/>
 <instance part="IC1" gate="G$1" x="149.86" y="76.2"/>
 <instance part="T1" gate="G$1" x="154.94" y="38.1"/>
+<instance part="U$3" gate="G$1" x="48.26" y="-2.54"/>
+<instance part="U$4" gate="G$1" x="45.72" y="-2.54"/>
+<instance part="U$5" gate="G$1" x="66.04" y="-5.08"/>
+<instance part="U$9" gate="G$1" x="68.58" y="-5.08"/>
+<instance part="U$10" gate="G$1" x="86.36" y="-5.08"/>
+<instance part="U$11" gate="G$1" x="88.9" y="-5.08"/>
+<instance part="U$12" gate="G$1" x="104.14" y="-5.08"/>
+<instance part="U$13" gate="G$1" x="106.68" y="-5.08"/>
+<instance part="U$14" gate="G$1" x="119.38" y="-5.08"/>
+<instance part="U$15" gate="G$1" x="121.92" y="-5.08"/>
+<instance part="U$16" gate="G$1" x="142.24" y="-5.08"/>
+<instance part="U$17" gate="G$1" x="144.78" y="-5.08"/>
+<instance part="U$18" gate="G$1" x="160.02" y="-5.08"/>
+<instance part="U$19" gate="G$1" x="162.56" y="-5.08"/>
+<instance part="JP1_LCD" gate="G$1" x="17.78" y="71.12" rot="R90"/>
+<instance part="U$20" gate="G$1" x="121.92" y="111.76"/>
+<instance part="POT1" gate="SW" x="160.02" y="101.6"/>
+<instance part="S1_POWER" gate="1" x="22.86" y="109.22" rot="R90"/>
 </instances>
 <busses>
@@
 <pinref part="J2" gate="G$1" pin="2"/>
 </segment>
-</net>
+<segment>
+<pinref part="SW1UP" gate="G$1" pin="S1"/>
+<pinref part="U$3" gate="G$1" pin="COM"/>
+</segment>
+<segment>
+<pinref part="SW1UP" gate="G$1" pin="S"/>
+<pinref part="U$4" gate="G$1" pin="COM"/>
+</segment>
+<segment>
+<pinref part="SW2RIGHT" gate="G$1" pin="S"/>
+<pinref part="U$5" gate="G$1" pin="COM"/>
+</segment>
+<segment>
+<pinref part="SW2RIGHT" gate="G$1" pin="S1"/>
+<pinref part="U$9" gate="G$1" pin="COM"/>
+</segment>
+<segment>
+<pinref part="SW3DOWN" gate="G$1" pin="S"/>
+<pinref part="U$10" gate="G$1" pin="COM"/>
+</segment>
+<segment>
+<pinref part="SW3DOWN" gate="G$1" pin="S1"/>
+<pinref part="U$11" gate="G$1" pin="COM"/>
+</segment>
+<segment>
+<pinref part="SW4LEFT" gate="G$1" pin="S"/>
+<pinref part="U$12" gate="G$1" pin="COM"/>
+</segment>
+<segment>
+<pinref part="SW4LEFT" gate="G$1" pin="S1"/>
+<pinref part="U$13" gate="G$1" pin="COM"/>
+</segment>
+<segment>
+<pinref part="SW5ABTN" gate="G$1" pin="S"/>
+<pinref part="U$14" gate="G$1" pin="COM"/>
+</segment>
+<segment>
+<pinref part="SW5ABTN" gate="G$1" pin="S1"/>
+<pinref part="U$15" gate="G$1" pin="COM"/>
+</segment>
+<segment>
+<pinref part="SW6BBTN" gate="G$1" pin="S"/>
+<pinref part="U$16" gate="G$1" pin="COM"/>
+</segment>
+<segment>
+<pinref part="SW6BBTN" gate="G$1" pin="S1"/>
+<pinref part="U$17" gate="G$1" pin="COM"/>
+</segment>
+<segment>
+<pinref part="SW7CBTN" gate="G$1" pin="S"/>
+<pinref part="U$18" gate="G$1" pin="COM"/>
+</segment>
+<segment>
+<pinref part="SW7CBTN" gate="G$1" pin="S1"/>
+<pinref part="U$19" gate="G$1" pin="COM"/>
+</segment>
+</net>
